Commit message: fix urdf

File: hunter_gazebo/urdf/camera.urdf.xacro (robot description, xacro)
@@ -1,4 +1,4 @@
 <!-- 摄像头相关的 xacro 文件 -->
-<robot name="my_camera" xmlns:xacro="http://wiki.ros.org/xacro">
+<robot name="camera" xmlns:xacro="http://wiki.ros.org/xacro">
     <!-- 摄像头属性 -->
     <xacro:property name="camera_length" value="0.01" /> <!-- 摄像头长度(x) -->

File: hunter_gazebo/urdf/hunter.urdf (robot description, URDF)
Before this commit: robot hunter, 10 links, 9 joints
Links:
- added link front_steer_link, mass 1.2963; visual sphere radius=0.0051
- added link rear_wheel_link, mass 1.2963; visual sphere radius=0.0051
- link base_link: mass 5 -> 17.26; geometry collision box size=0.3 0.3 0.06; visual box size=0.3 0.3 0.06
- link camera: geometry visual box size=0.01 0.02 0.03
- link front_left_wheel_link: mass 1 -> 0.2963; geometry collision mesh filename=package://hunter_gazebo/meshes/front_left_wheel_link.STL; visual mesh filename=package://hunter_gazebo/meshes/front_left_wheel_link.STL
- link front_right_wheel_link: mass 1 -> 0.2963; geometry collision mesh filename=package://hunter_gazebo/meshes/front_right_wheel_link.STL; visual mesh filename=package://hunter_gazebo/meshes/front_right_wheel_link.STL
- link front_steer_left_link: mass 0.01 -> 1.2963; geometry visual sphere radius=0.0051
- link front_steer_right_link: mass 0.01 -> 1.2963; geometry visual sphere radius=0.0051
- link left_rear_link: mass 1 -> 0.2963; geometry collision mesh filename=package://hunter_gazebo/meshes/front_left_wheel_link.STL; visual mesh filename=package://hunter_gazebo/meshes/front_left_wheel_link.STL
- link right_rear_link: mass 1 -> 0.2963; geometry collision mesh filename=package://hunter_gazebo/meshes/front_right_wheel_link.STL; visual mesh filename=package://hunter_gazebo/meshes/front_right_wheel_link.STL
- link support: geometry visual cylinder length=0.0925 radius=0.01
Joints:
- added joint front_steer_joint: type revolute, parent base_link, child front_steer_link, origin xyz=0.15 0 0 rpy=0 0 0, axis 0 0 1, limit lower=-0.69 upper=0.69 effort=0 velocity=0
- added joint rear_wheel_joint: type continuous, parent base_link, child rear_wheel_link, origin xyz=-0.15 0 0 rpy=0 0 0, axis 0 1 0
- joint camera2base_link: origin xyz=0.405 0.0 0.1125 -> xyz=0.145 0.0 0.045
- joint front_left_wheel_joint: origin xyz=0 0 -0.2 rpy=0 0 0 -> xyz=0 0 0 rpy=0 0 0
- joint front_right_wheel_joint: origin xyz=0 0 -0.2 rpy=0 0 0 -> xyz=0 0 0 rpy=0 0 0
- joint front_steer_left_joint: origin xyz=0.15 0.105 0.2 rpy=0 0 0 -> xyz=0.15 0.205 0 rpy=0 0 0
- joint front_steer_right_joint: origin xyz=0.15 -0.105 0.2 rpy=0 0 0 -> xyz=0.15 -0.205 0 rpy=0 0 0
- joint laser2support: origin xyz=0.0 0.0 0.15 -> xyz=0.0 0.0 0.07125000000000001
- joint left_rear_joint: origin xyz=-0.15 0.105 0 rpy=0 0 0 -> xyz=-0.15 0.21 0 rpy=0 0 0
- joint right_rear_joint: origin xyz=-0.15 -0.105 0 rpy=0 0 0 -> xyz=-0.15 -0.21 0 rpy=0 0 0
- joint support2base_link: origin xyz=0.0 0.0 0.1 -> xyz=0.0 0.0 0.03

File: hunter_gazebo/urdf/hunter.urdf.xacro (robot description, xacro)
@@ -1,6 +1,6 @@
 <!-- 组合小车底盘与摄像头与雷达 -->
 <robot name="hunter" xmlns:xacro="http://wiki.ros.org/xacro">
-    <xacro:include filename="h.urdf.xacro" />
-    <xacro:include filename="hunter_b.urdf.xacro" />
+    <xacro:include filename="head.urdf.xacro" />
+    <xacro:include filename="hunter_base.urdf.xacro" />
     <xacro:include filename="camera.urdf.xacro" />
     <xacro:include filename="laser.urdf.xacro" />

File: hunter_gazebo/urdf/hunter_base.urdf.xacro (robot description, xacro)
@@ -1,20 +1,20 @@
-<robot name="my_camera" xmlns:xacro="http://wiki.ros.org/xacro">
-    <xacro:include filename="head.xacro" />
-    <xacro:property name="length" value="0.8" />
-    <xacro:property name="width" value="0.4" />
-    <xacro:property name="high" value="0.2" />
-    <xacro:property name="base_mass" value="10" />
+<!-- 组合小车底盘与摄像头与雷达 -->
+<robot name="hunter_b" xmlns:xacro="http://wiki.ros.org/xacro">
+    <xacro:include filename="head.urdf.xacro" />
+    <xacro:property name="length" value="0.3" />
+    <xacro:property name="width" value="0.3" />
+    <xacro:property name="high" value="0.06" />
+    <xacro:property name="base_mass" value="17.26" />
     <xacro:property name="PI" value="3.141592653" />
     <xacro:property name="base_footprint_radius" value="0.001" /> <!-- base_footprint 半径  -->
-    <xacro:property name="wheel_radius" value="0.15" /><!-- 半径 -->
-    <xacro:property name="wheel_width" value="0.06" /><!-- 宽度 -->
-    <xacro:property name="wheel_m" value="2.5" />
-    <link name="base_footprint">
-      <visual>
-        <geometry>
-          <sphere radius="${base_footprint_radius}" />
-        </geometry>
-      </visual>
-    </link>
+    <xacro:property name="wheel_radius" value="0.0625" /><!-- 半径 -->
+    <xacro:property name="wheel_width" value="0.03" /><!-- 宽度 -->
+    <xacro:property name="wheel_m" value="0.2963" />
+    <gazebo>
+        <plugin name="gazebo_ros_control" filename="libgazebo_ros_control.so">
+        <robotSimType>steer_bot_hardware_gazebo/SteerBotHardwareGazebo</robotSimType>
+        <legacyModeNS>false</legacyModeNS>
+        </plugin>
+    </gazebo>
     <link name="base_link">
         <xacro:Box_inertial_matrix m="${base_mass}" l="${length}" w="${width}" h="${high}" xyz="0 0 0" rpy="0 0 0"/>
@@ -32,20 +32,24 @@
         </collision>
     </link>
-    <gazebo reference="base_link">
-        <material>Gazebo/Black</material>
-    </gazebo>
+    <!-- <link name="base_footprint">
+      <visual>
+        <geometry>
+          <sphere radius="${base_footprint_radius}" />
+        </geometry>
+      </visual>
+    </link>
     <joint name="base_link2base_footprint" type="fixed">
       <parent link="base_footprint" />
       <child link="base_link" />
       <origin xyz="0 0 ${wheel_radius - high / 2 }" />
-    </joint>
+    </joint> -->
     <!-- rear -->
-    <xacro:macro name="add_rear_wheels" params="name flag x y z xyz rpy"> <!--left 1--> <!--right -1-->
+    <xacro:macro name="add_rear_wheels" params="name flag x y z xyz rpy"> <!--left flag=1--> <!--right flag=-1-->
         <link name="${name}_rear_link">
-            <xacro:cylinder_inertial_matrix m="${wheel_m}" r="${wheel_radius}" h="${wheel_width}" xyz="${xyz}" rpy="${rpy}"/>
+            <xacro:cylinder_inertial_matrix m="${wheel_m}" r="${wheel_radius}" h="${wheel_width}" xyz="${xyz}" rpy="${PI/2} 0 0"/>
             <visual>
                 <origin xyz="${xyz}" rpy="${rpy}" />
                 <geometry>
-                    <cylinder radius="${wheel_radius}" length="${wheel_width}" />
+                    <mesh filename="package://hunter_gazebo/meshes/front_${name}_wheel_link.STL" />
                 </geometry>
                 <material name="black">
@@ -56,8 +60,11 @@
                 <origin xyz="${xyz}" rpy="${rpy}" />
                 <geometry>
-                    <cylinder radius="${wheel_radius}" length="${wheel_width}" />
+                    <mesh filename="package://hunter_gazebo/meshes/front_${name}_wheel_link.STL" />
                 </geometry>
             </collision>
         </link>
+        <gazebo reference="${name}_rear_link">
+            <material>Gazebo/Black</material>
+        </gazebo>
         <joint name="${name}_rear_joint" type="continuous">
             <origin xyz="${-x} ${flag * y} ${z}" rpy="0 0 0" />
@@ -75,17 +82,17 @@
         </gazebo>
     </xacro:macro>
-    <xacro:add_rear_wheels name="left" flag="1.0" x="0.3" y="0.33" z="0" xyz="0 0 0" rpy="${PI/2} 0 0"/>
-    <xacro:add_rear_wheels name="right" flag="-1.0" x="0.3" y="0.33" z="0" xyz="0 0 0" rpy="${PI/2} 0 0"/>
+    <xacro:add_rear_wheels name="left" flag="1.0" x="${length/2}" y="${width/2+0.06}" z="0" xyz="0 0 0" rpy="0 0 0"/>
+    <xacro:add_rear_wheels name="right" flag="-1.0" x="${length/2}" y="${width/2+0.06}" z="0" xyz="0 0 0" rpy="0 0 0"/>
     <!-- front -->
-    <xacro:property name="steer_radius" value="0.0051" /><!-- 半径 -->
-    <xacro:property name="steer_width" value="0.0051" /><!-- 宽度 -->
+    <xacro:property name="support_wheel_radius" value="0.025" />
+    <!-- too small will be errors since default controller param "P" is big-->
     <xacro:property name="steer_m" value="0.1" />
-    <xacro:macro name="add_front_wheels" params="name flag x y z xyz rpy"> <!--left 1--> <!--right -1-->
+    <xacro:macro name="add_front_wheels" params="name flag x y z xyz rpy"> <!--left flag=1--> <!--right flag=-1-->
         <link name="front_steer_${name}_link">
-            <xacro:cylinder_inertial_matrix m="${steer_m}" r="${steer_radius}" h="${steer_width}" xyz="0 0 0" rpy="0 0 0"/>
+            <xacro:sphere_inertial_matrix m="${steer_m}" r="${support_wheel_radius}"/>
             <visual>
-                <origin rpy="0 0 0"  xyz="0 0 0" />
+                <origin xyz="${xyz}" rpy="${rpy}" />
                 <geometry>
-                    <cylinder radius="${steer_radius}" length="${steer_width}" />
+                    <sphere radius="${support_wheel_radius}" />
                 </geometry>
                 <material name="black">
@@ -93,10 +100,4 @@
                 </material>
             </visual>
-            <!--collision>
-                <origin rpy="0 0 0"  xyz="0 0 0" />
-                <geometry>
-                    <cylinder radius="${steer_radius}" length="${steer_width}" />
-                </geometry>
-            </collision-->
         </link>
         <joint name="front_steer_${name}_joint" type="revolute">
@@ -108,9 +109,9 @@
         </joint>
         <link name="front_${name}_wheel_link">
-            <xacro:cylinder_inertial_matrix m="${wheel_m}" r="${wheel_radius}" h="${wheel_width}" xyz="${xyz}" rpy="${rpy}"/>
+            <xacro:cylinder_inertial_matrix m="${wheel_m}" r="${wheel_radius}" h="${wheel_width}" xyz="${xyz}" rpy="${PI/2} 0 0"/>
             <visual>
                 <origin xyz="${xyz}" rpy="${rpy}" />
                 <geometry>
-                    <cylinder radius="${wheel_radius}" length="${wheel_width}" />
+                    <mesh filename="package://hunter_gazebo/meshes/front_${name}_wheel_link.STL" />
                 </geometry>
                 <material name="black">
@@ -121,5 +122,5 @@
                 <origin xyz="${xyz}" rpy="${rpy}" />
                 <geometry>
-                    <cylinder radius="${wheel_radius}" length="${wheel_width}" />
+                    <mesh filename="package://hunter_gazebo/meshes/front_${name}_wheel_link.STL" />
                 </geometry>
             </collision>
@@ -131,15 +132,52 @@
             <axis xyz="0 1 0" />
         </joint>
-        <gazebo reference="front_steer_${name}_link">
+        <gazebo reference="front_${name}_wheel_link">
             <material>Gazebo/Red</material>
         </gazebo>
     </xacro:macro>
-    <xacro:add_front_wheels name="left" flag="1.0" x="0.3" y="0.33" z="0.2" xyz="0 0 0" rpy="${PI/2} 0 0"/>
-    <xacro:add_front_wheels name="right" flag="-1.0" x="0.3" y="0.33" z="0.2" xyz="0 0 0" rpy="${PI/2} 0 0"/>
-    <gazebo>
-        <plugin name="gazebo_ros_control" filename="libgazebo_ros_control.so">
-        <robotSimType>steer_bot_hardware_gazebo/SteerBotHardwareGazebo</robotSimType>
-        <legacyModeNS>false</legacyModeNS>
-        </plugin>
+    <xacro:add_front_wheels name="left" flag="1.0" x="${length/2}" y="${width/2+0.055}" z="0" xyz="0 0 0" rpy="0 0 0"/>
+    <xacro:add_front_wheels name="right" flag="-1.0" x="${length/2}" y="${width/2+0.055}" z="0" xyz="0 0 0" rpy="0 0 0"/>
+    <!-- for steer_drive_controller -->
+    <xacro:property name="drive_m" value="0.001" />
+    <xacro:property name="drive_r" value="0.01" />
+    <link name="front_steer_link">
+        <xacro:sphere_inertial_matrix m="${drive_m}" r="${drive_r}"/>
+        <visual>
+            <origin rpy="0 0 0"  xyz="0 0 0" />
+            <geometry>
+                <sphere radius="${drive_r}" />
+            </geometry>
+            <material name="black">
+                <color rgba="0.0 0.0 0.0 1.0" />
+            </material>
+        </visual>
+    </link>
+    <gazebo reference="front_steer_link">
+            <material>Gazebo/Red</material>
     </gazebo>
+    <joint name="front_steer_joint" type="revolute">
+        <origin xyz="${length/2} 0 0" rpy="0 0 0" />
+        <parent link="base_link" />
+        <child link="front_steer_link" />
+        <axis xyz="0 0 1" />
+        <limit lower="-0.69" upper="0.69" effort="0" velocity="0" />
+    </joint>
+    <link name="rear_wheel_link">
+        <xacro:sphere_inertial_matrix m="${drive_m}" r="${drive_r}"/>
+        <visual>
+            <origin rpy="0 0 0"  xyz="0 0 0" />
+            <geometry>
+                <sphere radius="${drive_r}" />
+            </geometry>
+            <material name="black">
+                <color rgba="0.0 0.0 0.0 1.0" />
+            </material>
+        </visual>
+    </link>
+    <joint name="rear_wheel_joint" type="continuous">
+        <origin xyz="-${length/2} 0 0" rpy="0 0 0" />
+        <parent link="base_link" />
+        <child link="rear_wheel_link" />
+        <axis xyz="0 1 0" />
+    </joint>
 </robot>
